File: untitled.brd (EAGLE design)
At the start: 89.3 x 82.9 mm, 116 parts, among them IC4 MCP23017SS, K2 351, Q1 S9013, U49 PC817X2NIP0F

Commit message: revisi PCB
Parts:
- removed TERMINAL-BLOCK10P1, TERMINAL-BLOCK10P2: (no value), terminal-blok10p:TERMINA-BLOK10P
- added AC1: (no value), pinhead:1X02
- added X1, X2: MSTBA8, con-phoenix-508:MSTBA8
- added X3, X4: MSTBA3, con-phoenix-508:MSTBA3
- added X5, X6: MSTBA2, con-phoenix-508:MSTBA2
- moved R52 199.2 mm to (51.4, 33.4), flipped to the bottom, turned to 270 degrees
- moved R51 196.0 mm to (54.1, 33.4), flipped to the bottom, turned to 270 degrees
- moved R98 177.4 mm to (60.2, 51.5), flipped to the bottom, turned to 90 degrees
- moved R106 172.6 mm to (64.9, 43.8), flipped to the bottom
- moved R97 169.1 mm to (57.3, 51.5), flipped to the bottom, turned to 90 degrees
- moved R105 168.1 mm to (64.9, 41.5), flipped to the bottom
- moved R104 163.9 mm to (64.9, 39.1), flipped to the bottom
- moved R64 161.0 mm to (54.4, 51.5), flipped to the bottom, turned to 90 degrees
- moved R103 159.8 mm to (65.0, 36.7), flipped to the bottom
- moved R63 152.8 mm to (51.4, 51.6), flipped to the bottom, turned to 90 degrees
- moved R62 144.7 mm to (48.3, 51.6), flipped to the bottom, turned to 90 degrees
- moved R61 136.8 mm to (45.1, 51.6), flipped to the bottom, turned to 90 degrees
- moved R60 129.3 mm to (42.2, 51.6), flipped to the bottom, turned to 90 degrees
- moved R59 125.7 mm to (41.0, 47.9), flipped to the bottom
- moved R58 122.6 mm to (41.1, 45.5), flipped to the bottom
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Connections:
- removed net GND_SYSTEM: TERMINAL-BLOCK10P2.9
- new net 24V+: AC1.1, X4.2
- new net 24V-: AC1.2, X4.1
- net +: now also X6.2; no longer TERMINAL-BLOCK10P1.P$1
- net -: now also X6.1; no longer TERMINAL-BLOCK10P1.11
- net A+: now also X5.1; no longer TERMINAL-BLOCK10P2.P$1
- net B-: now also X5.2; no longer TERMINAL-BLOCK10P2.11
- net COMM: now also X4.3; no longer TERMINAL-BLOCK10P2.10
- net COMMON: now also X3.2; no longer TERMINAL-BLOCK10P1.9
- net NC: now also X3.3
- net NO: now also X3.1; no longer TERMINAL-BLOCK10P1.10
- net P1: now also X1.8; no longer TERMINAL-BLOCK10P1.1
- net P10: now also X2.2; no longer TERMINAL-BLOCK10P2.2
- net P11: now also X2.3; no longer TERMINAL-BLOCK10P2.3
- net P12: now also X2.4; no longer TERMINAL-BLOCK10P2.4
- net P13: now also X2.5; no longer TERMINAL-BLOCK10P2.5
- net P14: now also X2.6; no longer TERMINAL-BLOCK10P2.6
- net P15: now also X2.7; no longer TERMINAL-BLOCK10P2.7
- net P16: now also X2.8; no longer TERMINAL-BLOCK10P2.8
- net P2: now also X1.7; no longer TERMINAL-BLOCK10P1.2
- net P3: now also X1.6; no longer TERMINAL-BLOCK10P1.3
- net P4: now also X1.5; no longer TERMINAL-BLOCK10P1.4
- net P5: now also X1.4; no longer TERMINAL-BLOCK10P1.5
- net P6: now also X1.3; no longer TERMINAL-BLOCK10P1.6
- net P7: now also X1.2; no longer TERMINAL-BLOCK10P1.7
- net P8: now also X1.1; no longer TERMINAL-BLOCK10P1.8
- net P9: now also X2.1; no longer TERMINAL-BLOCK10P2.1
Routing:
- net COMM: track 0.00 -> 425.1 mm, vias 0 -> 2
- net GND: track 0.00 -> 228.7 mm, vias 0 -> 3
- net VCC: track 0.00 -> 195.3 mm, vias 0 -> 1
- net OUT16: track 0.00 -> 114.9 mm, vias 0 -> 1
- net OUT15: track 0.00 -> 114.4 mm, vias 0 -> 1
- net SCL: track 0.00 -> 84.8 mm, vias 0 -> 1
- net SDA: track 0.00 -> 70.3 mm, vias 0 -> 2
- net OUT4: track 0.00 -> 68.4 mm, vias 0 -> 1
- net OUT3: track 0.00 -> 55.8 mm, vias 0 -> 1
- net OUT9: track 0.00 -> 54.2 mm, vias 0 -> 1
- net OUT10: track 0.00 -> 49.1 mm, vias 0 -> 1
- net N$101: track 0.00 -> 48.3 mm, vias 0 -> 1
- net OUT2: track 0.00 -> 48.2 mm, vias 0 -> 1
- net OUT1: track 0.00 -> 41.7 mm, vias 0 -> 1
- net OUT11: track 0.00 -> 35.8 mm, vias 0 -> 1
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Other:
- board size 89.3 x 82.9 mm -> 87.8 x 82.9 mm
- board text added: "24V"
- board text added: "GND"
- board text added: "RELAY"
- board text added: "RX"
- board text added: "SCL"
- board text added: "SDA"
- board text added: "TX"
- board text added: "VCC"
