File: untitled.brd (EAGLE design)
At the start: 87.8 x 82.9 mm, 121 parts, among them IC4 MCP23017SS, K2 351, Q1 S9013, U49 PC817X2NIP0F, X1 MSTBA8, X2 MSTBA8, X3 MSTBA3, X4 MSTBA3, X5 MSTBA2, X6 MSTBA2

Commit message: revisi .brd
Routing:
- net TX: track 31.8 -> 21.7 mm
Other:
- outline, holes or cut-outs redrawn
Changed lines of the file:
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@@
 <wire x1="88.7" y1="37.8" x2="88.7" y2="-0.1" width="0" layer="20"/>
 <wire x1="88.7" y1="-0.1" x2="1" y2="0" width="0" layer="20"/>
-<circle x="8.2" y="64.1" radius="1.5" width="0.005" layer="20"/>
+<circle x="9.0128" y="66.2336" radius="1.5" width="0.005" layer="20"/>
 <circle x="85.2" y="49.1" radius="1.5" width="0.005" layer="20"/>
 <circle x="85" y="33" radius="1.5" width="0.005" layer="20"/>
@@
 <wire x1="57.34" y1="52.44" x2="57.39" y2="52.49" width="0.2" layer="16"/>
 <wire x1="57.39" y1="52.49" x2="60.24" y2="52.49" width="0.2" layer="16"/>
-<wire x1="53.455" y1="46.686" x2="53.455" y2="47.155" width="0.2" layer="16"/>
-<wire x1="53.455" y1="47.155" x2="55.7" y2="49.4" width="0.2" layer="16"/>
-<wire x1="55.7" y1="49.4" x2="55.7" y2="52.09" width="0.2" layer="16"/>
+<wire x1="53.455" y1="46.686" x2="53.455" y2="47.4852" width="0.2" layer="16"/>
+<wire x1="53.455" y1="47.4852" x2="55.7" y2="49.7302" width="0.2" layer="16"/>
+<wire x1="55.7" y1="49.7302" x2="55.7" y2="52.09" width="0.2" layer="16"/>
 <wire x1="55.7" y1="52.09" x2="56.1" y2="52.49" width="0.2" layer="16"/>
 <wire x1="59.44" y1="32.33" x2="62.63" y2="32.33" width="0.2" layer="16"/>
@@
 <contactref element="TTL-RS1" pad="TX"/>
 <contactref element="SV2" pad="6"/>
-<wire x1="21.696875" y1="66.932809375" x2="21.696875" y2="63.996875" width="0.4064" layer="16"/>
-<wire x1="21.696875" y1="63.996875" x2="20.9" y2="63.2" width="0.4064" layer="16"/>
-<wire x1="20.9" y1="63.2" x2="13.7" y2="63.2" width="0.4064" layer="16"/>
-<wire x1="13.7" y1="63.2" x2="12.8" y2="64.1" width="0.4064" layer="16"/>
-<wire x1="12.8" y1="64.1" x2="12.8" y2="67.5" width="0.4064" layer="16"/>
-<wire x1="12.8" y1="67.5" x2="11.2" y2="69.1" width="0.4064" layer="16"/>
-<wire x1="11.2" y1="69.1" x2="5.5" y2="69.1" width="0.4064" layer="16"/>
-<wire x1="5.5" y1="69.1" x2="4.1" y2="67.7" width="0.4064" layer="16"/>
-<wire x1="4.1" y1="67.7" x2="4.1" y2="61.76" width="0.4064" layer="16"/>
+<wire x1="19.9008" y1="61.76" x2="4.1" y2="61.76" width="0.4064" layer="16"/>
+<wire x1="21.696875" y1="66.932809375" x2="21.696875" y2="63.556075" width="0.4064" layer="16"/>
+<wire x1="21.696875" y1="63.556075" x2="19.9008" y2="61.76" width="0.4064" layer="16"/>
 </signal>
 <signal name="RX">
